File: bf-021/bf-021.kicad_pcb (KiCad board)
At the start: 2 copper layers, 50 x 50 mm, 9 parts, among them J1 M-BUS

Commit message: V01L01
replace
Connections:
- J1 pad 1: GND -> /GPIO35
- J1 pad 10: /GPIO26 -> /GPIO19
- J1 pad 11: /GPIO18 -> +3V3
- J1 pad 12: +3V3 -> /GPIO18
- J1 pad 13: /GPIO3 -> /GPIO1
- J1 pad 14: /GPIO1 -> /GPIO3
- J1 pad 15: /GPIO16 -> /GPIO17
- J1 pad 16: /GPIO17 -> /GPIO16
- J1 pad 17: /GPIO21 -> /GPIO22
- J1 pad 18: /GPIO22 -> /GPIO21
- J1 pad 19: /GPIO2 -> /GPIO5
- J1 pad 2: /GPIO35 -> GND
- J1 pad 20: /GPIO5 -> /GPIO2
- J1 pad 21: /GPIO12 -> /GPIO13
- J1 pad 22: /GPIO13 -> /GPIO12
- J1 pad 23: /GPIO15 -> /GPIO0
- J1 pad 24: /GPIO0 -> /GPIO15
- J1 pad 25: VBUS -> /GPIO34
- J1 pad 26: /GPIO34 -> VBUS
- J1 pad 27: VBUS -> +5V
- J1 pad 28: +5V -> VBUS
- J1 pad 29: VBUS -> +BATT
- J1 pad 3: GND -> /GPIO36
- J1 pad 30: +BATT -> VBUS
- J1 pad 4: /GPIO36 -> GND
- J1 pad 5: GND -> /EN
- J1 pad 6: /EN -> GND
- J1 pad 7: /GPIO23 -> /GPIO25
- J1 pad 8: /GPIO25 -> /GPIO23
- J1 pad 9: /GPIO19 -> /GPIO26
Routing:
- net GND: track 24.5 -> 30.9 mm
- net VBUS: track 5.08 -> 6.90 mm

Commit message: V01L01
replace
Other:
- board text removed: "0"
- board text removed: "1"
- board text removed: "12"
- board text removed: "13"
- board text removed: "15"
- board text removed: "16"
- board text removed: "17"
- board text removed: "18"
- board text removed: "19"
- board text removed: "2"
- board text removed: "21"
- board text removed: "22"
- board text removed: "23"
- board text removed: "25"
- board text removed: "26"
- board text removed: "3"
- board text removed: "34"
- board text removed: "35"
- board text removed: "36"
- board text removed: "3V3"
- board text removed: "5"
- board text removed: "5V"
- board text removed: "BAT"
- board text removed: "EN"
- board text removed: "GND"
- board text removed: "HPWR"
